File: high_power_switch_controller_3x2.sch (KiCad schematic (older format))
At the start: 1 part

Commit message: hitfet -> high_power_switch.
Parts:
- MDB1: footprint hitfet_controller_3x2:MODULAR_DEVICE_BASE_3X2_MALE -> high_power_switch_controller_3x2:MODULAR_DEVICE_BASE_3X2_MALE
Changed lines of the file:
@@
 LIBS:contrib
 LIBS:valves
-LIBS:hitfet_controller_3x2
+LIBS:high_power_switch_controller_3x2
 LIBS:components
 EELAYER 26 0
@@
 encoding utf-8
 Sheet 1 1
-Title "hitfet_controller_3x2"
+Title "high_power_switch_controller_3x2"
 Date ""
 Rev "1.0"
@@
 F 0 "MDB1" H 2650 2547 60  0000 C CNN
 F 1 "MODULAR_DEVICE_BASE_3X2_MALE" H 2650 2441 60  0000 C CNN
-F 2 "hitfet_controller_3x2:MODULAR_DEVICE_BASE_3X2_MALE" H 600 1050 60  0001 C CNN
+F 2 "high_power_switch_controller_3x2:MODULAR_DEVICE_BASE_3X2_MALE" H 600 1050 60  0001 C CNN
 F 3 "" H 650 2750 60  0000 C CNN
 F 4 "digikey" H 600 1150 60  0001 C CNN "Vendor"

Commit message: Updated to v4.
Parts:
- MDB1: symbol MODULAR_DEVICE_BASE_3X2_MALE -> high_power_switch_controller_3x2:MODULAR_DEVICE_BASE_3X2_MALE
Connections:
- wire segments 8 -> 11
Changed lines of the file:
@@
-EESchema Schematic File Version 2
-LIBS:power
-LIBS:device
-LIBS:transistors
-LIBS:conn
-LIBS:linear
-LIBS:regul
-LIBS:74xx
-LIBS:cmos4000
-LIBS:adc-dac
-LIBS:memory
-LIBS:xilinx
-LIBS:microcontrollers
-LIBS:dsp
-LIBS:microchip
-LIBS:analog_switches
-LIBS:motorola
-LIBS:texas
-LIBS:intel
-LIBS:audio
-LIBS:interface
-LIBS:digital-audio
-LIBS:philips
-LIBS:display
-LIBS:cypress
-LIBS:siliconi
-LIBS:opto
-LIBS:atmel
-LIBS:contrib
-LIBS:valves
-LIBS:high_power_switch_controller_3x2
-LIBS:components
+EESchema Schematic File Version 4
 EELAYER 26 0
 EELAYER END
@@
 $EndDescr
 $Comp
-L MODULAR_DEVICE_BASE_3X2_MALE MDB1
+L high_power_switch_controller_3x2:MODULAR_DEVICE_BASE_3X2_MALE MDB1
 U 1 1 589B6745
 P 2650 1550
@@
 $EndComp
 $Comp
-L VDD #PWR?
+L power:VDD #PWR?
 U 1 1 589B67C3
 P 1350 750
@@
 $EndComp
 $Comp
-L PWR_FLAG #FLG?
+L power:PWR_FLAG #FLG?
 U 1 1 589B67D9
 P 1100 750
@@
 	1100 750  1100 800
 Wire Wire Line
-	1100 800  1400 800
+	1100 800  1350 800
 Wire Wire Line
 	1350 750  1350 800
 Connection ~ 1350 800
 $Comp
-L GND #PWR?
+L power:GND #PWR?
 U 1 1 589B67FE
 P 700 950
@@
 $EndComp
 $Comp
-L PWR_FLAG #FLG?
+L power:PWR_FLAG #FLG?
 U 1 1 589B6835
 P 700 750
@@
 $EndComp
 Wire Wire Line
-	700  750  700  950
+	700  750  700  900
 Wire Wire Line
 	700  900  1400 900
@@
 NoConn ~ 3900 2300
 $Comp
-L VEE #PWR?
+L power:VEE #PWR?
 U 1 1 589B69B5
 P 4450 800
@@
 $EndComp
 $Comp
-L PWR_FLAG #FLG?
+L power:PWR_FLAG #FLG?
 U 1 1 589B69CA
 P 4750 800
@@
 	4750 800  4750 900
 Wire Wire Line
-	4750 900  3900 900
+	4750 900  4450 900
 Wire Wire Line
 	4450 800  4450 900
 Connection ~ 4450 900
+Wire Wire Line
+	1350 800  1400 800
+Wire Wire Line
+	700  900  700  950
+Wire Wire Line
+	4450 900  3900 900
 $EndSCHEMATC
